Commit message: feat: move to origin

File: hiro-urdf/robot.urdf (robot description, URDF)
Before this commit: robot hiro-urdf3, 22 links, 21 joints
Links:
- removed link base_link
Joints:
- removed joint base_to_torso
- joint left_ankle_pitch: origin xyz=-8.67362e-17 -0.111702 -5.55112e-17 rpy=3.14159 -3.35505e-30 -1.16573e-15 -> xyz=-8.67362e-17 -0.111702 -6.59195e-17 rpy=3.14159 -3.35505e-30 -1.16573e-15
- joint left_ankle_roll: origin xyz=-0.02558 6.93889e-18 0.0235 rpy=1.89327e-29 1.5708 0 -> xyz=-0.02558 0 0.0235 rpy=1.89327e-29 1.5708 0
- joint left_hip_pitch: origin xyz=0.0235 -2.77556e-17 -0.02558 rpy=-1.11022e-16 1.5708 0 -> xyz=0.0235 -2.60209e-17 -0.02558 rpy=-1.11022e-16 1.5708 0
- joint left_hip_roll: origin xyz=-0.0335 3.56659e-14 0.032 rpy=-1.5708 -1.30562e-13 1.5708 -> xyz=-0.0335 3.56451e-14 0.032 rpy=-1.5708 -1.30562e-13 1.5708
- joint left_hip_yaw: origin xyz=0.19561 0.0108657 0.272566 rpy=3.14159 1.14304e-14 -1.5708 -> xyz=0.0495 -0.0149156 0.0210065 rpy=3.14159 1.14304e-14 -1.5708
- joint left_knee: origin xyz=-6.41848e-16 -0.134 2.77556e-17 rpy=-1.26218e-29 -3.51852e-31 -6.52256e-15 -> xyz=-6.42715e-16 -0.134 4.16334e-17 rpy=-1.26218e-29 -3.51852e-31 -6.52256e-15
- joint left_shoulder_pitch: origin xyz=0.218397 0.0065975 0.412866 rpy=1.5708 -1.05839e-14 1.5708 -> xyz=0.0722867 -0.0191838 0.161307 rpy=1.5708 -1.05839e-14 1.5708
- joint neck_yaw: origin xyz=0.146197 -0.0189018 0.436266 rpy=2.15281e-13 -1.12084e-14 1.5708 -> xyz=8.67185e-05 -0.0446832 0.184707 rpy=2.15281e-13 -1.12084e-14 1.5708
- joint right_ankle_pitch: origin xyz=-1.11022e-16 0.111702 2.77556e-17 rpy=-3.14159 -1.44182e-29 -6.31382e-14 -> xyz=-1.10155e-16 0.111702 2.08167e-17 rpy=-3.14159 -1.44182e-29 -6.31382e-14
- joint right_ankle_roll: origin xyz=-0.02558 -4.43135e-15 0.0235 rpy=2.06085e-15 1.5708 0 -> xyz=-0.02558 -4.44089e-15 0.0235 rpy=2.06085e-15 1.5708 0
- joint right_hip_pitch: origin xyz=0.0235 2.77556e-17 -0.02558 rpy=-1.88064e-27 1.5708 0 -> xyz=0.0235 4.68375e-17 -0.02558 rpy=-1.88064e-27 1.5708 0
- joint right_hip_yaw: origin xyz=0.0966103 0.0108641 0.272566 rpy=3.14159 1.14304e-14 -1.5708 -> xyz=-0.0495 -0.0149172 0.0210065 rpy=3.14159 1.14304e-14 -1.5708
- joint right_knee: origin xyz=-6.21031e-16 0.134 2.77556e-17 rpy=2.08167e-16 7.21645e-16 1.53223e-14 -> xyz=-6.16694e-16 0.134 4.16334e-17 rpy=2.08167e-16 7.21645e-16 1.53223e-14
- joint right_shoulder_pitch: origin xyz=0.0738235 0.0065975 0.412866 rpy=1.5708 1.08614e-14 -1.5708 -> xyz=-0.0722867 -0.0191838 0.161307 rpy=1.5708 1.08614e-14 -1.5708

Commit message: fix: missing mass

File: hiro-urdf/robot.urdf (robot description, URDF)
Before this commit: robot hiro-urdf, 21 links, 20 joints
Links:
- link foot_left_2: mass 0.13801 -> 0.273181
- link foot_right_1: mass 0.288767 -> 0.292396
- link foot_right_2: mass 0.13801 -> 0.273181
Joints:
- joint left_ankle_roll: origin xyz=-0.02558 0 0.0235 rpy=1.89327e-29 1.5708 0 -> xyz=-0.02558 0 0.0235 rpy=1.96989e-29 1.5708 0

Commit message: fix: axis inv orientation

File: hiro-urdf/robot.urdf (robot description, URDF)
Before this commit: robot hiro-urdf3, 21 links, 20 joints
Joints:
- joint left_ankle_pitch: origin xyz=-8.67362e-17 -0.111702 -6.59195e-17 rpy=3.14159 -3.35505e-30 -1.16573e-15 -> xyz=-8.67362e-17 0.111702 6.59195e-17 rpy=-4.35572e-28 3.35505e-30 1.16573e-15
- joint left_elbow: origin xyz=-0.09951 0.0205971 0.0156 rpy=-1.5708 1.5708 0 -> xyz=-0.09951 -0.0205971 -0.0156 rpy=1.5708 -1.5708 0
- joint left_hip_pitch: limit lower=-1.1781 upper=1.9635 effort=6 velocity=6.6 -> lower=-1.9635 upper=1.1781 effort=6 velocity=6.6; origin xyz=0.0235 -2.60209e-17 -0.02558 rpy=-1.11022e-16 1.5708 0 -> xyz=0.0235 2.60209e-17 0.02558 rpy=-1.11022e-16 -1.5708 0
- joint left_hip_roll: origin xyz=-0.0335 3.56451e-14 0.032 rpy=-1.5708 -1.30562e-13 1.5708 -> xyz=-0.0335 -3.56451e-14 -0.032 rpy=-1.5708 1.30562e-13 -1.5708
- joint left_hip_yaw: limit lower=-0.785398 upper=1.5708 effort=6 velocity=6.6 -> lower=-1.5708 upper=0.785398 effort=6 velocity=6.6; origin xyz=0.0495 -0.0149156 0.0210065 rpy=3.14159 1.14304e-14 -1.5708 -> xyz=0.0495 -0.0149156 0.0210065 rpy=-2.1517e-13 1.14304e-14 -1.5708
- joint left_knee: limit lower=-0.785398 upper=0.785398 effort=6 velocity=6.6 -> lower=-2.35619 upper=2.35619 effort=6 velocity=6.6; origin xyz=-6.42715e-16 -0.134 4.16334e-17 rpy=-1.26218e-29 -3.51852e-31 -6.52256e-15 -> xyz=-6.42715e-16 0.134 -4.16334e-17 rpy=-1.26218e-29 3.51852e-31 6.52256e-15
- joint left_shoulder_roll: limit lower=-0.785398 upper=2.35619 effort=6 velocity=6.6 -> lower=-2.35619 upper=0.785398 effort=6 velocity=6.6; origin xyz=-0.0205 -0.0147498 0.0268034 rpy=-0 1.5708 0 -> xyz=-0.0205 -0.0147498 0.0268034 rpy=-3.14159 1.5708 0
- joint right_ankle_pitch: origin xyz=-1.10155e-16 0.111702 2.08167e-17 rpy=-3.14159 -1.44182e-29 -6.31382e-14 -> xyz=-1.10155e-16 0.111702 2.08167e-17 rpy=2.44616e-28 -1.44182e-29 -6.31382e-14
- joint right_ankle_roll: origin xyz=-0.02558 -4.44089e-15 0.0235 rpy=2.06085e-15 1.5708 0 -> xyz=-0.02558 4.44089e-15 -0.0235 rpy=-3.14159 -1.5708 0
- joint right_elbow: origin xyz=-0.0205971 0.09951 0.0256 rpy=-5.89437e-27 -1.5708 0 -> xyz=-0.0205971 -0.09951 -0.0256 rpy=-5.89437e-27 1.5708 0
- joint right_hip_pitch: origin xyz=0.0235 4.68375e-17 -0.02558 rpy=-1.88064e-27 1.5708 0 -> xyz=0.0235 -4.68375e-17 0.02558 rpy=3.14159 -1.5708 0
- joint right_hip_roll: origin xyz=-0.0335 -3.55965e-14 0.032 rpy=1.5708 1.23013e-13 -1.5708 -> xyz=-0.0335 3.55965e-14 -0.032 rpy=1.5708 -1.23013e-13 1.5708
- joint right_hip_yaw: limit lower=-1.5708 upper=0.785398 effort=6 velocity=6.6 -> lower=-0.785398 upper=1.5708 effort=6 velocity=6.6; origin xyz=-0.0495 -0.0149172 0.0210065 rpy=3.14159 1.14304e-14 -1.5708 -> xyz=-0.0495 -0.0149172 0.0210065 rpy=-2.15281e-13 1.14304e-14 -1.5708
- joint right_shoulder_pitch: origin xyz=-0.0722867 -0.0191838 0.161307 rpy=1.5708 1.08614e-14 -1.5708 -> xyz=-0.0722867 -0.0191838 0.161307 rpy=-1.5708 1.08614e-14 -1.5708
- joint right_shoulder_roll: limit lower=-2.35619 upper=0.785398 effort=6 velocity=6.6 -> lower=-0.785398 upper=2.35619 effort=6 velocity=6.6; origin xyz=0.0205 -0.0147498 0.0268034 rpy=1.5708 1.30895e-13 -1.5708 -> xyz=0.0205 0.0147498 -0.0268034 rpy=1.5708 -1.30895e-13 1.5708

Commit message: feat: add frames

File: hiro-urdf/robot.urdf (robot description, URDF)
Before this commit: robot hiro-urdf, 21 links, 20 joints
Links:
- added link left_foot, mass 1e-9; visual sphere radius=0.01
- added link right_foot, mass 1e-9; visual sphere radius=0.01
- added link trunk, mass 1e-9; visual sphere radius=0.01
Joints:
- removed joint neck_pitch
- removed joint neck_yaw
- added joint head_pitch: type revolute, parent neck, child head, origin xyz=5e-07 -0.0205 0.037 rpy=-1.5708 -1.5708 0, axis 0 0 1, limit lower=-1.5708 upper=0.392699 effort=6 velocity=6.6
- added joint head_yaw: type revolute, parent torso_kidsize25, child neck, origin xyz=8.67185e-05 -0.0446832 0.184707 rpy=2.15281e-13 -1.12084e-14 1.5708, axis 0 0 1, limit lower=-3.14159 upper=3.14159 effort=6 velocity=6.6
- added joint left_foot_frame: type revolute, parent foot_left_5, child left_foot, origin xyz=0.0 0.032 0.03 rpy=0 -1.5708 1.5708, axis 0 0 1, limit lower=0.0 upper=0.0 effort=0.0 velocity=0.0
- added joint right_foot_frame: type revolute, parent foot_right_5, child right_foot, origin xyz=0.0 -0.032 0.03 rpy=0 -1.5708 -1.5708, axis 0 0 1, limit lower=0.0 upper=0.0 effort=0.0 velocity=0.0
- added joint trunk_frame: type fixed, parent torso_kidsize25, child trunk, origin xyz=0.0 0.0 0.02 rpy=0 0 -1.5708, axis 0 0 1
